Commit message: added six_wheel_steering_msgs

File: argo_mini_urdf_6w_drive/urdf/main.xacro (robot description, xacro)
@@ -40,12 +40,15 @@
     <xacro:macro name="gazebo_wheel" params="link">
         <gazebo reference="${link}">
-            <mu1>1.2</mu1>
-            <mu2>1.2</mu2>
+            <mu1>0.2</mu1>
+            <mu2>0.2</mu2>
             <fdir1>1 0 0</fdir1>
-            <maxContacts>1</maxContacts>
+            <maxContacts>20</maxContacts>
             <minDepth>0.005</minDepth>
             <gravity>true</gravity>
             <material>Gazebo/Black</material>
         </gazebo>
+    </xacro:macro>
+    <xacro:macro name="turn_dynamics">
+        <dynamics damping="0.05" friction="0.1"/>
     </xacro:macro>
     <link name="drive_base">
@@ -141,10 +144,11 @@
                 link="front_left_turn_link"/>
         <axis
-                xyz="0 0 1"/>
+                xyz="0 0 -1"/>
         <limit
-                lower="-3.14"
-                upper="3.14"
+                lower="-1.57"
+                upper="1.57"
                 effort="100"
                 velocity="3.14"/>
+        <xacro:turn_dynamics/>
     </joint>
     <link name="front_left_wheel_link">
@@ -189,5 +193,5 @@
                 link="front_left_wheel_link"/>
         <axis
-                xyz="0 0 -1"/>
+                xyz="0 0 1"/>
     </joint>
     <link name="front_right_turn_link">
@@ -240,10 +244,11 @@
                 link="front_right_turn_link"/>
         <axis
-                xyz="0 0 1"/>
+                xyz="0 0 -1"/>
         <limit
-                lower="-3.14"
-                upper="3.14"
+                lower="-1.57"
+                upper="1.57"
                 effort="100"
                 velocity="3.14"/>
+        <xacro:turn_dynamics/>
     </joint>
     <link name="front_right_wheel_link">
@@ -339,10 +344,11 @@
                 link="mid_left_turn_link"/>
         <axis
-                xyz="0 0 1"/>
+                xyz="0 0 -1"/>
         <limit
-                lower="-3.14"
-                upper="3.14"
+                lower="-1.57"
+                upper="1.57"
                 effort="100"
                 velocity="3.14"/>
+        <xacro:turn_dynamics/>
     </joint>
     <link name="mid_left_wheel_link">
@@ -387,5 +393,5 @@
                 link="mid_left_wheel_link"/>
         <axis
-                xyz="0 0 -1"/>
+                xyz="0 0 1"/>
     </joint>
     <link name="mid_right_turn_link">
@@ -438,10 +444,11 @@
                 link="mid_right_turn_link"/>
         <axis
-                xyz="0 0 1"/>
+                xyz="0 0 -1"/>
         <limit
-                lower="-3.14"
-                upper="3.14"
+                lower="-1.57"
+                upper="1.57"
                 effort="100"
                 velocity="3.14"/>
+        <xacro:turn_dynamics/>
     </joint>
     <link name="mid_right_wheel_link">
@@ -537,10 +544,11 @@
                 link="rear_left_turn_link"/>
         <axis
-                xyz="0 0 1"/>
+                xyz="0 0 -1"/>
         <limit
-                lower="-3.14"
-                upper="3.14"
+                lower="-1.57"
+                upper="1.57"
                 effort="100"
                 velocity="3.14"/>
+        <xacro:turn_dynamics/>
     </joint>
     <link name="rear_left_wheel_link">
@@ -585,5 +593,5 @@
                 link="rear_left_wheel_link"/>
         <axis
-                xyz="0 0 -1"/>
+                xyz="0 0 1"/>
     </joint>
     <link name="rear_right_turn_link">
@@ -636,10 +644,11 @@
                 link="rear_right_turn_link"/>
         <axis
-                xyz="0 0 1"/>
+                xyz="0 0 -1"/>
         <limit
-                lower="-3.14"
-                upper="3.14"
+                lower="-1.57"
+                upper="1.57"
                 effort="100"
                 velocity="3.14"/>
+        <xacro:turn_dynamics/>
     </joint>
     <link name="rear_right_wheel_link">
