Commit message: added rplidar and front camera link

File: argo_mini_urdf_podstawa/urdf/argo_mini_urdf_podstawa.xacro (robot description, xacro)
@@ -96,4 +96,36 @@
                 velocity="3.14"/>
     </joint>
+     <link
+    name="front_camera">
+  </link>
+  <joint
+    name="front_camera_joint"
+    type="fixed">
+    <origin
+      xyz="0.29213 -0.0061284 -0.03"
+      rpy="-1.5708 0 -1.5708" />
+    <parent
+      link="base_link" />
+    <child
+      link="front_camera" />
+    <axis
+      xyz="0 0 0" />
+  </joint>
+  <link
+    name="rp_lidar_a1">
+  </link>
+  <joint
+    name="rp_lidar_a1_joint"
+    type="fixed">
+    <origin
+      xyz="0.23107 -0.0049901 -0.095067"
+      rpy="-3.1416 0 0" />
+    <parent
+      link="base_link" />
+    <child
+      link="rp_lidar_a1" />
+    <axis
+      xyz="0 0 0" />
+  </joint>
     <xacro:gazebo_corpse link="base_link"/>
     <xacro:property name="modules_config_file" value="$(find argo_mini_urdf_podstawa)/config/modules.yaml"/>

Commit message: added lidar and front camera

File: argo_mini_urdf_podstawa/urdf/argo_mini_urdf_podstawa.xacro (robot description, xacro)
@@ -80,12 +80,10 @@
     </link>
     <joint name="base_link_to_peripheral_base"
-            type="fixed">
+           type="fixed">
         <origin
                 xyz="0.19495 -0.0061284 0.0063061"
                 rpy="0 0 0"/>
-        <parent
-                link="base_link"/>
-        <child
-                link="peripheral_base"/>
+        <parent link="base_link"/>
+        <child link="peripheral_base"/>
         <axis
                 xyz="0 0 0"/>
@@ -96,36 +94,33 @@
                 velocity="3.14"/>
     </joint>
-     <link
-    name="front_camera">
-  </link>
-  <joint
-    name="front_camera_joint"
-    type="fixed">
-    <origin
-      xyz="0.29213 -0.0061284 -0.03"
-      rpy="-1.5708 0 -1.5708" />
-    <parent
-      link="base_link" />
-    <child
-      link="front_camera" />
-    <axis
-      xyz="0 0 0" />
-  </joint>
-  <link
-    name="rp_lidar_a1">
-  </link>
-  <joint
-    name="rp_lidar_a1_joint"
-    type="fixed">
-    <origin
-      xyz="0.23107 -0.0049901 -0.095067"
-      rpy="-3.1416 0 0" />
-    <parent
-      link="base_link" />
-    <child
-      link="rp_lidar_a1" />
-    <axis
-      xyz="0 0 0" />
-  </joint>
+    <link name="front_camera"/>
+    <joint name="front_camera_joint"
+            type="fixed">
+        <origin
+                xyz="0.29213 -0.0061284 -0.03"
+                rpy="0 0 0"
+        />
+        <!--                rpy="-1.5708 0 -1.5708"-->
+        <parent
+                link="base_link"/>
+        <child
+                link="front_camera"/>
+        <axis
+                xyz="0 0 0"/>
+    </joint>
+    <link name="rp_lidar_a1"/>
+    <joint
+            name="rp_lidar_a1_joint"
+            type="fixed">
+        <origin
+                xyz="0.23107 -0.0049901 -0.095067"
+                rpy="-3.1416 0 0"/>
+        <parent
+                link="base_link"/>
+        <child
+                link="rp_lidar_a1"/>
+        <axis
+                xyz="0 0 0"/>
+    </joint>
     <xacro:gazebo_corpse link="base_link"/>
     <xacro:property name="modules_config_file" value="$(find argo_mini_urdf_podstawa)/config/modules.yaml"/>
@@ -140,3 +135,76 @@
         </plugin>
     </gazebo>
+    <gazebo reference="front_camera">
+        <material>Gazebo/Green</material>
+        <sensor type="camera" name="front_camera">
+            <update_rate>30.0</update_rate>
+            <camera name="front">
+                <horizontal_fov>1.3962634</horizontal_fov>
+                <image>
+                    <width>1920</width>
+                    <height>1080</height>
+                    <format>R8G8B8</format>
+                </image>
+                <clip>
+                    <near>0.1</near>
+                    <far>300</far>
+                </clip>
+                <noise>
+                    <type>gaussian</type>
+                    <mean>0.0</mean>
+                    <stddev>0.00</stddev>
+                </noise>
+            </camera>
+            <plugin name="camera_controller" filename="libgazebo_ros_camera.so">
+                <alwaysOn>true</alwaysOn>
+                <updateRate>0.0</updateRate>
+                <cameraName>/front</cameraName>
+                <imageTopicName>image_raw</imageTopicName>
+                <cameraInfoTopicName>camera_info</cameraInfoTopicName>
+                <frameName>front_camera</frameName>
+                <hackBaseline>0.07</hackBaseline>
+                <distortionK1>0.0</distortionK1>
+                <distortionK2>0.0</distortionK2>
+                <distortionK3>0.0</distortionK3>
+                <distortionT1>0.0</distortionT1>
+                <distortionT2>0.0</distortionT2>
+            </plugin>
+        </sensor>
+    </gazebo>
+    <gazebo reference="rp_lidar_a1">
+        <material>Gazebo/Blue</material>
+        <sensor type="ray" name="head_hokuyo_sensor">
+            <pose>0 0 0 0 0 0</pose>
+            <visualize>true</visualize>
+            <update_rate>30</update_rate>
+            <ray>
+                <scan>
+                    <horizontal>
+                        <samples>720</samples>
+                        <resolution>1</resolution>
+                        <min_angle>-1.</min_angle>
+                        <max_angle>1.</max_angle>
+                    </horizontal>
+                </scan>
+                <range>
+                    <min>0.10</min>
+                    <max>15.0</max>
+                    <resolution>0.01</resolution>
+                </range>
+                <noise>
+                    <type>gaussian</type>
+                    <!-- Noise parameters based on published spec for Hokuyo laser
+                         achieving "+-30mm" accuracy at range < 10m.  A mean of 0.0m and
+                         stddev of 0.01m will put 99.7% of samples within 0.03m of the true
+                         reading. -->
+                    <mean>0.0</mean>
+                    <stddev>0.01</stddev>
+                </noise>
+            </ray>
+            <plugin name="gazebo_ros_head_hokuyo_controller" filename="libgazebo_ros_laser.so">
+                <topicName>/laser/scan</topicName>
+                <frameName>rp_lidar_a1</frameName>
+            </plugin>
+        </sensor>
+    </gazebo>
 </robot>

Commit message: tested with controllers on

File: argo_mini_urdf_podstawa/urdf/argo_mini_urdf_podstawa.xacro (robot description, xacro)
@@ -95,4 +95,5 @@
     </joint>
     <link name="front_camera"/>
+    <link name="front_camera_z"/>
     <joint name="front_camera_joint"
             type="fixed">
@@ -106,4 +107,17 @@
         <child
                 link="front_camera"/>
+        <axis
+                xyz="0 0 0"/>
+    </joint>
+    <joint name="front_camera_joint_z"
+            type="fixed">
+        <origin
+                xyz="0.29213 -0.0061284 -0.03"
+                rpy="-1.5708 0 -1.5708"
+        />
+        <parent
+                link="base_link"/>
+        <child
+                link="front_camera_z"/>
         <axis
                 xyz="0 0 0"/>

Commit message: urdf configuration with args

File: argo_mini_urdf_podstawa/urdf/argo_mini_urdf_podstawa.xacro (robot description, xacro)
@@ -138,9 +138,11 @@
     </joint>
     <xacro:gazebo_corpse link="base_link"/>
-    <xacro:property name="modules_config_file" value="$(find argo_mini_urdf_podstawa)/config/modules.yaml"/>
-    <xacro:property name="modules_config" value="${load_yaml(modules_config_file)}"/>
-    <xacro:include filename="$(find ${modules_config['drive']})/urdf/main.xacro"/>
-    <xacro:if value="${modules_config['peripheral'] != ''}">
-        <xacro:include filename="$(find ${modules_config['peripheral']})/urdf/main.xacro"/>
+    <xacro:arg name="drive" default="argo_mini_urdf_6w_drive"/>
+    <xacro:arg name="peripheral" default=""/>
+    <xacro:property name="drive_pkg_name" value="$(arg drive)"/>
+    <xacro:include filename="$(find ${drive_pkg_name})/urdf/main.xacro"/>
+    <xacro:if value="$(eval peripheral != '')">
+        <xacro:property name="peripheral_pkg_name" value="$(arg peripheral)"/>
+        <xacro:include filename="$(find ${peripheral_pkg_name})/urdf/main.xacro"/>
     </xacro:if>
     <gazebo>

Commit message: new peripheral added

File: argo_mini_urdf_podstawa/urdf/argo_mini_urdf_podstawa.xacro (robot description, xacro)
@@ -60,8 +60,8 @@
             <inertia
                     ixx="1e-3"
-                    ixy="1e-3"
-                    ixz="1e-3"
+                    ixy="0"
+                    ixz="0"
                     iyy="1e-3"
-                    iyz="1e-3"
+                    iyz="0"
                     izz="1e-3"/>
         </inertial>
@@ -69,5 +69,5 @@
             <origin xyz="0 0 0" rpy="0 0 0"/>
             <geometry>
-                <cylinder length="1e-3" radius="1e-3"/>
+                <cylinder length="1e-4" radius="1e-4"/>
             </geometry>
         </visual>
@@ -75,5 +75,5 @@
             <origin xyz="0 0 0" rpy="0 0 0"/>
             <geometry>
-                <cylinder length="1e-3" radius="1e-3"/>
+                <cylinder length="1e-4" radius="1e-4"/>
             </geometry>
         </collision>
@@ -86,11 +86,4 @@
         <parent link="base_link"/>
         <child link="peripheral_base"/>
-        <axis
-                xyz="0 0 0"/>
-        <limit
-                lower="-3.14"
-                upper="3.14"
-                effort="100"
-                velocity="3.14"/>
     </joint>
     <link name="front_camera"/>

Commit message: minor changes

File: argo_mini_urdf_podstawa/urdf/argo_mini_urdf_podstawa.xacro (robot description, xacro)
@@ -6,5 +6,5 @@
         </gazebo>
     </xacro:macro>
-    <link name="dummy"/>
+    <link name="base_footprint"/>
     <link
             name="base_link">
@@ -47,7 +47,8 @@
         </collision>
     </link>
-    <joint name="dummy_joint" type="fixed">
-        <parent link="dummy"/>
+    <joint name="base_to_footprint" type="fixed">
+        <parent link="base_footprint"/>
         <child link="base_link"/>
+        <origin xyz="0 0 0.2" rpy="0 0 0"/>
     </joint>
     <link name="peripheral_base">

Commit message: zed-wrapper remove, lidar on robot less samples, testing gmapping

File: argo_mini_urdf_podstawa/urdf/argo_mini_urdf_podstawa.xacro (robot description, xacro)
@@ -121,6 +121,7 @@
             name="rp_lidar_a1_joint"
             type="fixed">
-        <origin
-                xyz="0.23107 -0.0049901 -0.095067"
+<!--        xyz="0.23107 -0.0049901 -0.095067"-->
+        <origin
+                xyz="0.23107 -0.0049901 0.05"
                 rpy="-3.1416 0 0"/>
         <parent
@@ -191,5 +192,5 @@
                 <scan>
                     <horizontal>
-                        <samples>4000</samples>
+                        <samples>500</samples>
                         <resolution>1</resolution>
                         <min_angle>-3.14.</min_angle>
